Commit message: Updated visuals for glados

File: glados_description/urdf/glados.urdf.xacro (robot description, xacro)
@@ -3,5 +3,5 @@
     <xacro:include filename="$(find z1_description)/xacro/robot.xacro"/>
     <link name="shop"/>
-    <joint name="shop_link" type="fixed">
+    <joint name="shop_joint" type="fixed">
         <origin xyz="0 0 0" rpy="3.14159 0 0" />
         <parent link="shop"/>
@@ -25,3 +25,39 @@
     />
     </xacro:zed_camera>
+    <link name="head_link">
+        <visual>
+            <geometry>
+                <mesh filename="package://glados_description/meshes/g_head.dae"/>
+            </geometry>
+        </visual>
+    </link>
+    <joint name="head_joint" type="fixed">
+        <origin xyz="0 0 0" rpy="0 0 0" />
+        <parent link="link06"/>
+        <child link="head_link"/>
+    </joint>
+    <link name="midsection_link">
+        <visual>
+            <geometry>
+                <mesh filename="package://glados_description/meshes/g_mid.dae"/>
+            </geometry>
+        </visual>
+    </link>
+    <joint name="midsection_joint" type="fixed">
+        <origin xyz="0 0 0" rpy="0 0 0" />
+        <parent link="link03"/>
+        <child link="midsection_link"/>
+    </joint>
+    <link name="upper_link">
+        <visual>
+            <geometry>
+                <mesh filename="package://glados_description/meshes/g_upper.dae"/>
+            </geometry>
+        </visual>
+    </link>
+    <joint name="upper_joint" type="fixed">
+        <origin xyz="0 0 0" rpy="0 0 0" />
+        <parent link="link02"/>
+        <child link="upper_link"/>
+    </joint>
 </robot>

Commit message: Update to urdf

File: glados_description/urdf/glados.urdf.xacro (robot description, xacro)
@@ -13,5 +13,5 @@
     <xacro:arg name="cam_pos_x"     default="-0.5" />
     <xacro:arg name="cam_pos_y"     default="0.0" />
-    <xacro:arg name="cam_pos_z"     default="0.5" />
+    <xacro:arg name="cam_pos_z"     default="1.0" />
     <xacro:arg name="cam_roll"      default="3.14159" />
     <xacro:arg name="cam_pitch"     default="0.0" />
@@ -61,3 +61,15 @@
         <child link="upper_link"/>
     </joint>
+    <link name="eye_link" />
+    <joint name="eye_joint" type="fixed">
+        <origin xyz="0.32 0 0.07" rpy="0 -0.2 0" />
+        <parent link="link06"/>
+        <child link="eye_link"/>
+    </joint>
+    <link name="view_link" />
+    <joint name="view_joint" type="fixed">
+        <origin xyz="0 0 0.4" rpy="0 0 0" />
+        <parent link="world"/>
+        <child link="view_link"/>
+    </joint>
 </robot>

Commit message: Update to urdf and watcher to make movement nice

File: glados_description/urdf/glados.urdf.xacro (robot description, xacro)
@@ -69,5 +69,5 @@
     <link name="view_link" />
     <joint name="view_joint" type="fixed">
-        <origin xyz="0 0 0.4" rpy="0 0 0" />
+        <origin xyz="0 0 0.55" rpy="0 0 0" />
         <parent link="world"/>
         <child link="view_link"/>
